Commit message: reverting change of gripper_link in robotiq URDF

File: dumbo_description/urdf/robotiq/robotiq_hand.xacro (robot description, xacro)
@@ -7,5 +7,5 @@
   <joint name="robotiq_base_joint" type="fixed">
     <origin xyz = "0.0 0.0 0.33" rpy="${PI/2} 0.0 0.0" />
-    <parent link="right_arm_gripper_link"/>
+    <parent link="right_arm_7_link"/>
     <child link="robotiq_palm"/>
   </joint>
