Commit message: changed names of F/T sensor links and frames to *_ft_sensor (before: _FT_sensor)

File: dumbo_description/urdf/lwa/lwa.urdf.xacro (robot description, xacro)
@@ -236,11 +236,11 @@
       </collision>
     </link>
-    <!-- ==================== FT sensor ==================== -->
-    <joint name="${name}_FT_joint" type="fixed" >
-      <origin xyz="0.0 0.0 ${FT_sensor_distance}" rpy="0.0 0.0 0.0" />
+    <!-- ==================== F/T sensor ==================== -->
+    <joint name="${name}_ft_joint" type="fixed" >
+      <origin xyz="0.0 0.0 ${ft_sensor_distance}" rpy="0.0 0.0 0.0" />
       <parent link="${name}_7_link" />
-      <child link="${name}_FT_sensor" />
-    </joint>
-    <link name="${name}_FT_sensor">
+      <child link="${name}_ft_sensor" />
+    </joint>
+    <link name="${name}_ft_sensor">
       <inertial>
 	<origin xyz="0.0 0.0 0.0" rpy="0.0 0.0 0.0" />

File: dumbo_description/urdf/lwa/lwa_common.xacro (robot description, xacro)
@@ -44,5 +44,5 @@
   <property name="PRL80_radius" value="0.045" />
   <property name="PRL80_length" value="0.17" />
-  <!-- FT sensor distance from joint 7-->
-  <property name="FT_sensor_distance" value="0.219848"/>
+  <!-- F/T sensor distance from joint 7-->
+  <property name="ft_sensor_distance" value="0.219848"/>
 </robot>

Commit message: added *_arm_gripper_link to URDFs for compliance with Moveit

File: dumbo_description/urdf/lwa/lwa.urdf.xacro (robot description, xacro)
@@ -52,5 +52,5 @@
 	<origin xyz="0 0 ${-DUMBO_LINK1_LENGTH/2 + middle_plate_length_x/4 - PRL100_radius/2 + 0.02}" rpy="0 0 0" />
 	<geometry>
-	  <cylinder radius="${PRL100_radius+0.02}" length="${PRL100_length+0.02}"/>
+	  <cylinder radius="${PRL100_radius}" length="${PRL100_length}"/>
 	</geometry>
       </collision>
@@ -82,5 +82,5 @@
 	<origin xyz="0 0 0" rpy="0 0 0" />
 	<geometry>
-	  <cylinder radius="${PRL100_radius+0.02}" length="${PRL100_length+0.02}"/>
+	  <cylinder radius="${PRL100_radius}" length="${PRL100_length}"/>
 	</geometry>
       </collision>
@@ -112,5 +112,5 @@
 	<origin xyz="0 0 ${-DUMBO_DH_D_3/2}" rpy="0 0 0" />
 	<geometry>
-	  <cylinder radius="${PRL100_radius+0.02}" length="${PRL100_length+0.05}"/>
+	  <cylinder radius="${PRL100_radius}" length="${PRL100_length}"/>
 	</geometry>
       </collision>
@@ -142,5 +142,5 @@
 	<origin xyz="0 0 0" rpy="0 0 0" />
 	<geometry>
-	  <cylinder radius="${PRL100_radius+0.02}" length="${PRL100_length+0.02}"/>
+	  <cylinder radius="${PRL100_radius}" length="${PRL100_length}"/>
 	</geometry>
       </collision>
@@ -172,5 +172,5 @@
 	<origin xyz="0 0 ${-DUMBO_DH_D_5/2 - PRL80_radius/2 + PRL100_radius/2}" rpy="0 0 0" />
 	<geometry>
-	  <cylinder radius="${PRL80_radius+0.02}" length="${PRL80_length}"/>
+	  <cylinder radius="${PRL80_radius}" length="${PRL80_length}"/>
 	</geometry>
       </collision>
@@ -202,5 +202,5 @@
 	<origin xyz="0 0 0" rpy="0 0 0" />
 	<geometry>
-	  <cylinder radius="${PRL80_radius+0.02}" length="${PRL80_length+0.02}"/>
+	  <cylinder radius="${PRL80_radius}" length="${PRL80_length}"/>
 	</geometry>
       </collision>
@@ -232,5 +232,5 @@
 	<origin xyz="0 0 ${DUMBO_TOOL_LENGTH/2 + PRL80_radius/2 - PG70_length_z/2 - PG70_finger_length_z/2}" rpy="0 0 0"/>
 	<geometry>
-	  <cylinder radius="${PRL80_radius+0.02}" length="${PRL80_length}"/>
+	  <cylinder radius="${PRL80_radius}" length="${PRL80_length}"/>
 	</geometry>
       </collision>
@@ -258,8 +258,14 @@
 	<origin xyz="0.0 0.0 0.03" rpy="0.0 0.0 0.0"/>
 	<geometry>
-	  <cylinder radius="${PRL80_radius+0.02}" length="0.03"/>
-	</geometry>
-      </collision>
-    </link>
+	  <cylinder radius="${PRL80_radius}" length="0.03"/>
+	</geometry>
+      </collision>
+    </link>
+    <!-- ==================== Gripper link ==================== -->
+    <joint name="${name}_gripper_base_joint" type="fixed" >
+      <origin xyz="0.0 0.0 0.0" rpy="0.0 0.0 0.0" />
+      <parent link="${name}_7_link" />
+      <child link="${name}_gripper_link" />
+    </joint>
   </xacro:macro>
 </robot>

File: dumbo_description/urdf/robotiq/robotiq_hand.xacro (robot description, xacro)
@@ -7,5 +7,5 @@
   <joint name="robotiq_base_joint" type="fixed">
     <origin xyz = "0.0 0.0 0.33" rpy="${PI/2} 0.0 0.0" />
-    <parent link="right_arm_7_link"/>
+    <parent link="right_arm_gripper_link"/>
     <child link="robotiq_palm"/>
   </joint>

Commit message: reverting gripper_link change in URDF

File: dumbo_description/urdf/lwa/lwa.urdf.xacro (robot description, xacro)
@@ -262,10 +262,4 @@
       </collision>
     </link>
-    <!-- ==================== Gripper link ==================== -->
-    <joint name="${name}_gripper_base_joint" type="fixed" >
-      <origin xyz="0.0 0.0 0.0" rpy="0.0 0.0 0.0" />
-      <parent link="${name}_7_link" />
-      <child link="${name}_gripper_link" />
-    </joint>
   </xacro:macro>
 </robot>

Commit message: fixed max joint velocities

File: dumbo_description/urdf/lwa/lwa.urdf.xacro (robot description, xacro)
@@ -33,5 +33,5 @@
       <parent link="${name}_0_link" />
       <child link="${name}_1_link" />
-      <limit effort="370" velocity="${30*PI/180}" lower="${-180*PI/180}" upper="${180*PI/180}"/>
+      <limit effort="370" velocity="${24*PI/180}" lower="${-180*PI/180}" upper="${180*PI/180}"/>
       <safety_controller k_position="100" k_velocity="10" soft_lower_limit="${-180*PI/180 + 2*PI/180}" soft_upper_limit="${180*PI/180 - 2*PI/180}" />
     </joint>
@@ -63,5 +63,5 @@
       <parent link="${name}_1_link" />
       <child link="${name}_2_link" />
-      <limit effort="370" velocity="${30*PI/180}" lower="${-120*PI/180}" upper="${120*PI/180}"/>
+      <limit effort="370" velocity="${24*PI/180}" lower="${-120*PI/180}" upper="${120*PI/180}"/>
       <safety_controller k_position="100" k_velocity="10" soft_lower_limit="${-120*PI/180 + 2*PI/180}" soft_upper_limit="${120*PI/180 - 2*PI/180}" />
     </joint>
@@ -93,5 +93,5 @@
       <parent link="${name}_2_link" />
       <child link="${name}_3_link" />
-      <limit effort="370" velocity="${30*PI/180}" lower="${-PI}" upper="${PI}"/>
+      <limit effort="370" velocity="${24*PI/180}" lower="${-PI}" upper="${PI}"/>
       <safety_controller k_position="100" k_velocity="10" soft_lower_limit="${-PI + 2*PI/180}" soft_upper_limit="${PI - 2*PI/180}" />
     </joint>
@@ -123,5 +123,5 @@
       <parent link="${name}_3_link" />
       <child link="${name}_4_link" />
-      <limit effort="370" velocity="${30*PI/180}" lower="${-120*PI/180}" upper="${120*PI/180}"/>
+      <limit effort="370" velocity="${24*PI/180}" lower="${-120*PI/180}" upper="${120*PI/180}"/>
       <safety_controller k_position="100" k_velocity="10" soft_lower_limit="${-120*PI/180 + 2*PI/180}" soft_upper_limit="${120*PI/180 - 2*PI/180}" />
     </joint>
@@ -153,5 +153,5 @@
       <parent link="${name}_4_link" />
       <child link="${name}_5_link" />
-      <limit effort="370" velocity="${30*PI/180}" lower="${-PI}" upper="${PI}"/>
+      <limit effort="370" velocity="${25*PI/180}" lower="${-PI}" upper="${PI}"/>
       <safety_controller k_position="100" k_velocity="10" soft_lower_limit="${-PI + 2*PI/180}" soft_upper_limit="${PI - 2*PI/180}" />
     </joint>
@@ -183,5 +183,5 @@
       <parent link="${name}_5_link" />
       <child link="${name}_6_link" />
-      <limit effort="370" velocity="${30*PI/180}" lower="${-112*PI/180}" upper="${112*PI/180}"/>
+      <limit effort="370" velocity="${25*PI/180}" lower="${-112*PI/180}" upper="${112*PI/180}"/>
       <safety_controller k_position="100" k_velocity="10" soft_lower_limit="${-112*PI/180 + 2*PI/180}" soft_upper_limit="${112*PI/180 - 2*PI/180}" />
     </joint>
@@ -213,5 +213,5 @@
       <parent link="${name}_6_link" />
       <child link="${name}_7_link" />
-      <limit effort="370" velocity="${38*PI/180}" lower="${-PI-3*PI/180}" upper="${PI+3*PI/180}"/>
+      <limit effort="370" velocity="${25*PI/180}" lower="${-PI-3*PI/180}" upper="${PI+3*PI/180}"/>
       <safety_controller k_position="100" k_velocity="10" soft_lower_limit="${-PI - PI/180}" soft_upper_limit="${PI + PI/180}" />
     </joint>

Commit message: beefed up max joint velocities

File: dumbo_description/urdf/lwa/lwa.urdf.xacro (robot description, xacro)
@@ -33,5 +33,5 @@
       <parent link="${name}_0_link" />
       <child link="${name}_1_link" />
-      <limit effort="370" velocity="${24*PI/180}" lower="${-180*PI/180}" upper="${180*PI/180}"/>
+      <limit effort="370" velocity="${38*PI/180}" lower="${-180*PI/180}" upper="${180*PI/180}"/>
       <safety_controller k_position="100" k_velocity="10" soft_lower_limit="${-180*PI/180 + 2*PI/180}" soft_upper_limit="${180*PI/180 - 2*PI/180}" />
     </joint>
@@ -63,5 +63,5 @@
       <parent link="${name}_1_link" />
       <child link="${name}_2_link" />
-      <limit effort="370" velocity="${24*PI/180}" lower="${-120*PI/180}" upper="${120*PI/180}"/>
+      <limit effort="370" velocity="${38*PI/180}" lower="${-120*PI/180}" upper="${120*PI/180}"/>
       <safety_controller k_position="100" k_velocity="10" soft_lower_limit="${-120*PI/180 + 2*PI/180}" soft_upper_limit="${120*PI/180 - 2*PI/180}" />
     </joint>
@@ -93,5 +93,5 @@
       <parent link="${name}_2_link" />
       <child link="${name}_3_link" />
-      <limit effort="370" velocity="${24*PI/180}" lower="${-PI}" upper="${PI}"/>
+      <limit effort="370" velocity="${38*PI/180}" lower="${-PI}" upper="${PI}"/>
       <safety_controller k_position="100" k_velocity="10" soft_lower_limit="${-PI + 2*PI/180}" soft_upper_limit="${PI - 2*PI/180}" />
     </joint>
@@ -123,5 +123,5 @@
       <parent link="${name}_3_link" />
       <child link="${name}_4_link" />
-      <limit effort="370" velocity="${24*PI/180}" lower="${-120*PI/180}" upper="${120*PI/180}"/>
+      <limit effort="370" velocity="${38*PI/180}" lower="${-120*PI/180}" upper="${120*PI/180}"/>
       <safety_controller k_position="100" k_velocity="10" soft_lower_limit="${-120*PI/180 + 2*PI/180}" soft_upper_limit="${120*PI/180 - 2*PI/180}" />
     </joint>
@@ -153,5 +153,5 @@
       <parent link="${name}_4_link" />
       <child link="${name}_5_link" />
-      <limit effort="370" velocity="${25*PI/180}" lower="${-PI}" upper="${PI}"/>
+      <limit effort="370" velocity="${39.9*PI/180}" lower="${-PI}" upper="${PI}"/>
       <safety_controller k_position="100" k_velocity="10" soft_lower_limit="${-PI + 2*PI/180}" soft_upper_limit="${PI - 2*PI/180}" />
     </joint>
@@ -183,5 +183,5 @@
       <parent link="${name}_5_link" />
       <child link="${name}_6_link" />
-      <limit effort="370" velocity="${25*PI/180}" lower="${-112*PI/180}" upper="${112*PI/180}"/>
+      <limit effort="370" velocity="${39.9*PI/180}" lower="${-112*PI/180}" upper="${112*PI/180}"/>
       <safety_controller k_position="100" k_velocity="10" soft_lower_limit="${-112*PI/180 + 2*PI/180}" soft_upper_limit="${112*PI/180 - 2*PI/180}" />
     </joint>
@@ -213,5 +213,5 @@
       <parent link="${name}_6_link" />
       <child link="${name}_7_link" />
-      <limit effort="370" velocity="${25*PI/180}" lower="${-PI-3*PI/180}" upper="${PI+3*PI/180}"/>
+      <limit effort="370" velocity="${39.9*PI/180}" lower="${-PI-3*PI/180}" upper="${PI+3*PI/180}"/>
       <safety_controller k_position="100" k_velocity="10" soft_lower_limit="${-PI - PI/180}" soft_upper_limit="${PI + PI/180}" />
     </joint>
