Commit message: updated accelerometer calibration

File: dumbo_description/urdf/accelerometer/accelerometer.urdf.xacro (robot description, xacro)
@@ -9,5 +9,5 @@
     <!-- ==================== Accelerometer ==================== -->
     <joint name="${name}_joint" type="fixed" >
-      <origin xyz="0.0 -0.098 0.0" rpy="-1.5452 -0.0353 0.0295"/>
+      <origin xyz="0.0 -0.098 0.0" rpy="-1.5617 -0.0358 0.035"/>
       <parent link="${parent}" />
       <child link="${name}" />

Commit message: updated accelerometer calibration

File: dumbo_description/urdf/accelerometer/accelerometer.urdf.xacro (robot description, xacro)
@@ -9,5 +9,5 @@
     <!-- ==================== Accelerometer ==================== -->
     <joint name="${name}_joint" type="fixed" >
-      <origin xyz="0.0 -0.098 0.0" rpy="-1.5617 -0.0358 0.035"/>
+      <origin xyz="0.0 -0.098 0.0" rpy="-1.5332 -0.0259 0.0291"/>
       <parent link="${parent}" />
       <child link="${name}" />

Commit message: corrected accelerometer calibration

File: dumbo_description/urdf/accelerometer/accelerometer.urdf.xacro (robot description, xacro)
@@ -9,5 +9,5 @@
     <!-- ==================== Accelerometer ==================== -->
     <joint name="${name}_joint" type="fixed" >
-      <origin xyz="0.0 -0.098 0.0" rpy="-1.5332 -0.0259 0.0291"/>
+      <origin xyz="0.0 -0.098 0.0" rpy="-1.5240 -0.0367 0.0175"/>
       <parent link="${parent}" />
       <child link="${name}" />
