Commit message: switched acceloremeter to imu in urdf files

File: dumbo_description/robots/dumbo.urdf.xacro (robot description, xacro)
@@ -17,5 +17,5 @@
   <xacro:include filename="$(find dumbo_description)/urdf/platform/platform.urdf.xacro" />
   <xacro:include filename="$(find dumbo_description)/urdf/torso/torso.urdf.xacro" />
-  <xacro:include filename="$(find dumbo_description)/urdf/accelerometer/accelerometer.urdf.xacro" />
+  <xacro:include filename="$(find dumbo_description)/urdf/imu/imu.urdf.xacro" />
   <xacro:include filename="$(find dumbo_description)/urdf/lwa/lwa.urdf.xacro" />
   <xacro:include filename="$(find dumbo_description)/urdf/gripper/gripper.urdf.xacro" />
@@ -27,6 +27,6 @@
     <origin xyz = "0.0 0.06 ${platform_length_z + torso_length/2}" rpy="0.0 0.0 0.0" />
   </xacro:dumbo_torso>
-  <!-- Accelerometer -->
-  <xacro:dumbo_accelerometer name="accelerometer" parent="arm_base_link" />
+  <!-- Imu -->
+  <xacro:dumbo_imu name="imu" parent="arm_base_link" />
   <!-- Schunk LWA -->
   <xacro:dumbo_lwa name="right_arm" parent="arm_base_link" reflect="1" />

File: dumbo_description/robots/dumbo_2grippers.urdf.xacro (robot description, xacro)
@@ -17,5 +17,5 @@
   <xacro:include filename="$(find dumbo_description)/urdf/platform/platform.urdf.xacro" />
   <xacro:include filename="$(find dumbo_description)/urdf/torso/torso.urdf.xacro" />
-  <xacro:include filename="$(find dumbo_description)/urdf/accelerometer/accelerometer.urdf.xacro" />
+  <xacro:include filename="$(find dumbo_description)/urdf/imu/imu.urdf.xacro" />
   <xacro:include filename="$(find dumbo_description)/urdf/lwa/lwa.urdf.xacro" />
   <xacro:include filename="$(find dumbo_description)/urdf/gripper/gripper.urdf.xacro" />
@@ -27,6 +27,6 @@
     <origin xyz = "0.0 0.06 ${platform_length_z + torso_length/2}" rpy="0.0 0.0 0.0" />
   </xacro:dumbo_torso>
-  <!-- Accelerometer -->
-  <xacro:dumbo_accelerometer name="accelerometer" parent="arm_base_link" />
+  <!-- Imu -->
+  <xacro:dumbo_imu name="imu" parent="arm_base_link" />
   <!-- Schunk LWA -->
   <xacro:dumbo_lwa name="right_arm" parent="arm_base_link" reflect="1" />

File: dumbo_description/robots/dumbo_robotiq.urdf.xacro (robot description, xacro)
@@ -17,5 +17,5 @@
   <xacro:include filename="$(find dumbo_description)/urdf/platform/platform.urdf.xacro" />
   <xacro:include filename="$(find dumbo_description)/urdf/torso/torso.urdf.xacro" />
-  <xacro:include filename="$(find dumbo_description)/urdf/accelerometer/accelerometer.urdf.xacro" />
+  <xacro:include filename="$(find dumbo_description)/urdf/imu/imu.urdf.xacro" />
   <xacro:include filename="$(find dumbo_description)/urdf/lwa/lwa.urdf.xacro" />
   <xacro:include filename="$(find dumbo_description)/urdf/gripper/gripper.urdf.xacro" />
@@ -28,6 +28,6 @@
     <origin xyz = "0.0 0.06 ${platform_length_z + torso_length/2}" rpy="0.0 0.0 0.0" />
   </xacro:dumbo_torso>
-  <!-- Accelerometer -->
-  <xacro:dumbo_accelerometer name="accelerometer" parent="arm_base_link" />
+  <!-- Imu -->
+  <xacro:dumbo_imu name="imu" parent="arm_base_link" />
   <!-- Schunk LWA -->
   <xacro:dumbo_lwa name="right_arm" parent="arm_base_link" reflect="1" />

File: dumbo_description/robots/dumbo_sdh.urdf.xacro (robot description, xacro)
@@ -17,5 +17,5 @@
   <xacro:include filename="$(find dumbo_description)/urdf/platform/platform.urdf.xacro" />
   <xacro:include filename="$(find dumbo_description)/urdf/torso/torso.urdf.xacro" />
-  <xacro:include filename="$(find dumbo_description)/urdf/accelerometer/accelerometer.urdf.xacro" />
+  <xacro:include filename="$(find dumbo_description)/urdf/imu/imu.urdf.xacro" />
   <xacro:include filename="$(find dumbo_description)/urdf/lwa/lwa.urdf.xacro" />
   <xacro:include filename="$(find dumbo_description)/urdf/gripper/gripper.urdf.xacro" />
@@ -28,6 +28,6 @@
     <origin xyz = "0.0 0.06 ${platform_length_z + torso_length/2}" rpy="0.0 0.0 0.0" />
   </xacro:dumbo_torso>
-  <!-- Accelerometer -->
-  <xacro:dumbo_accelerometer name="accelerometer" parent="arm_base_link" />
+  <!-- Imu -->
+  <xacro:dumbo_imu name="imu" parent="arm_base_link" />
   <!-- Schunk LWA -->
   <xacro:dumbo_lwa name="right_arm" parent="arm_base_link" reflect="1" />

File: dumbo_description/urdf/imu/imu.urdf.xacro (robot description, xacro)
@@ -4,8 +4,8 @@
        xmlns:interface="http://playerstage.sourceforge.net/gazebo/xmlschema/#interface"
        xmlns:xacro="http://ros.org/wiki/xacro">
-  <!-- macro for setting up the reference frame of the accelerometer (Phidgets 1056 IMU)
+  <!-- macro for setting up the reference frame of the IMU (Phidgets 1056 IMU)
        reflect = 1 for right arm, -1 for the left arm -->
-  <xacro:macro name="dumbo_accelerometer" params="name parent">
-    <!-- ==================== Accelerometer ==================== -->
+  <xacro:macro name="dumbo_imu" params="name parent">
+    <!-- ==================== IMU ==================== -->
     <joint name="${name}_joint" type="fixed" >
       <origin xyz="0.0 -0.098 0.0" rpy="-1.5240 -0.0367 0.0175"/>
