Commit message: lowered masses to 0.01 of arm and gripper links to allow gazebo velocity control simulation to work, increased gripper max vel

File: dumbo_description/urdf/gripper/gripper.urdf.xacro (robot description, xacro)
@@ -14,5 +14,5 @@
       <parent link="${parent}" />
       <child link="${name}_${prefix}_finger_link" />
-      <limit effort="370" velocity="0.01" lower="0.0" upper="0.03"/>
+      <limit effort="370" velocity="0.1" lower="0.0" upper="0.03"/>
       <safety_controller k_position="100" k_velocity="10" soft_lower_limit="0.001" soft_upper_limit="${0.03-0.001}" />
     </joint>
@@ -20,5 +20,5 @@
       <inertial>
 	<origin xyz="0 ${reflect*PG70_finger_length_y/2} ${PG70_finger_length_z/2}" rpy="0 0 0" />
-	<mass value="1.0" />
+	<mass value="0.01" />
 	<inertia ixx="0.01" ixy="0" ixz="0" iyy="0.01" iyz="0" izz="0.01" />
       </inertial>
@@ -49,5 +49,5 @@
       <inertial>
 	<origin xyz="0 0 ${-PG70_finger_length_z - PG70_length_z/2}" rpy="0 0 0" />
-	<mass value="1.0" />
+	<mass value="0.01" />
 	<inertia ixx="0.01" ixy="0" ixz="0" iyy="0.01" iyz="0" izz="0.01" />
       </inertial>

File: dumbo_description/urdf/lwa/lwa.urdf.xacro (robot description, xacro)
@@ -18,5 +18,5 @@
       <inertial>
 	<origin xyz="0 0 0" rpy="0 0 0"/>
-	<mass value="1.0"/>
+	<mass value="0.01"/>
 	<inertia ixx="0.01" ixy="0" ixz="0" iyy="0.01" iyz="0" izz="0.01" />
       </inertial>
@@ -41,5 +41,5 @@
       <inertial>
 	<origin xyz="0 0 ${-DUMBO_LINK1_LENGTH/2 + middle_plate_length_x/4 - PRL100_radius/2}" rpy="0.0 0.0 0.0"/>
-	<mass value="1.0"/>
+	<mass value="0.01"/>
 	<inertia ixx="0.01" ixy="0" ixz="0" iyy="0.01" iyz="0" izz="0.01" />
       </inertial>
@@ -71,5 +71,5 @@
       <inertial>
 	<origin xyz="0 0 0" rpy="0 0 0"/>
-	<mass value="1.0"/>
+	<mass value="0.01"/>
 	<inertia ixx="0.01" ixy="0" ixz="0" iyy="0.01" iyz="0" izz="0.01" />
       </inertial>
@@ -101,5 +101,5 @@
       <inertial>
 	<origin xyz="0 0 ${-DUMBO_DH_D_3/2}" rpy="0 0 0"/>
-	<mass value="1.0"/>
+	<mass value="0.01"/>
 	<inertia ixx="0.01" ixy="0" ixz="0" iyy="0.01" iyz="0" izz="0.01" />
       </inertial>
@@ -131,5 +131,5 @@
       <inertial>
 	<origin xyz="0 0 0" rpy="0 0 0"/>
-	<mass value="1.0"/>
+	<mass value="0.01"/>
 	<inertia ixx="0.01" ixy="0" ixz="0" iyy="0.01" iyz="0" izz="0.01" />
       </inertial>
@@ -161,5 +161,5 @@
       <inertial>
 	<origin xyz="0 0 ${-DUMBO_DH_D_5/2 - PRL80_radius/2 + PRL100_radius/2}" rpy="0 0 0"/>
-	<mass value="1.0"/>
+	<mass value="0.01"/>
 	<inertia ixx="0.01" ixy="0" ixz="0" iyy="0.01" iyz="0" izz="0.01" />
       </inertial>
@@ -191,5 +191,5 @@
       <inertial>
 	<origin xyz="0 0 0" rpy="0 0 0"/>
-	<mass value="1.0"/>
+	<mass value="0.01"/>
 	<inertia ixx="0.01" ixy="0" ixz="0" iyy="0.01" iyz="0" izz="0.01" />
       </inertial>
@@ -221,5 +221,5 @@
       <inertial>
 	<origin xyz="0 0 ${DUMBO_TOOL_LENGTH/2 + PRL80_radius/2 - PG70_length_z/2 - PG70_finger_length_z/2}" rpy="0 0 0" />
-	<mass value="1.0"/>
+	<mass value="0.01"/>
 	<inertia ixx="0.01" ixy="0" ixz="0" iyy="0.01" iyz="0" izz="0.01" />
       </inertial>
@@ -247,5 +247,5 @@
       <inertial>
 	<origin xyz="0.0 0.0 0.0" rpy="0.0 0.0 0.0" />
-	<mass value="1.0"/>
+	<mass value="0.01"/>
 	<inertia ixx="0.01" ixy="0" ixz="0" iyy="0.01" iyz="0" izz="0.01" />
       </inertial>

Commit message: incremented gripper joint pos limit due to optoforce sensors

File: dumbo_description/urdf/gripper/gripper.urdf.xacro (robot description, xacro)
@@ -14,5 +14,6 @@
       <parent link="${parent}" />
       <child link="${name}_${prefix}_finger_link" />
-      <limit effort="370" velocity="0.1" lower="0.0" upper="0.03"/>
+      <!-- setting lower position limit to 0.0155 because of the optoforce -->
+      <limit effort="370" velocity="0.1" lower="0.0155" upper="0.03"/>
       <safety_controller k_position="100" k_velocity="10" soft_lower_limit="0.001" soft_upper_limit="${0.03-0.001}" />
     </joint>
